File: TMC2209_Camera_Slider/PCB_Files/TMC2209_Camera_Slider_PCB_revB.brd (EAGLE design)
At the start: 100 x 70 mm, 114 parts, among them J1 1X2-3.5MM, J2 1X2-3.5MM, X1 REMBRANDT-ELECTRONICS---JST-X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, X2 REMBRANDT-ELECTRONICS---JST-X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

Commit message: move label
Parts:
- moved PLABEL0 0.50 mm to (88.0, 19.0)
Changed lines of the file:
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@@
 </element>
 <element name="U$1" library="microbuilder" package="ADAFRUIT_9MM" value="" x="15" y="37" smashed="yes" rot="R90"/>
-<element name="PLABEL0" library="pinguin" package="PLABEL0" value="" x="88.5" y="19" smashed="yes"/>
+<element name="PLABEL0" library="pinguin" package="PLABEL0" value="" x="88" y="19" smashed="yes"/>
 <element name="PLABEL2" library="pinguin" package="PLABEL2" value="" x="61.5" y="25" smashed="yes"/>
 <element name="PLABEL3" library="pinguin" package="PLABEL3" value="" x="34" y="25" smashed="yes"/>

Commit message: minor nudging
Parts:
- moved PLABEL203 0.50 mm to (17.5, 38.5)
Routing:
- net ENC_B: track 67.7 -> 68.4 mm
Changed lines of the file:
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@@
 <element name="PLABEL201" library="pinguin" package="PLABEL201" value="" x="49.5" y="45" smashed="yes" rot="R90"/>
 <element name="PLABEL202" library="pinguin" package="PLABEL202" value="" x="13" y="65" smashed="yes"/>
-<element name="PLABEL203" library="pinguin" package="PLABEL203" value="" x="18" y="38.5" smashed="yes" rot="MR0"/>
+<element name="PLABEL203" library="pinguin" package="PLABEL203" value="" x="17.5" y="38.5" smashed="yes" rot="MR0"/>
 <element name="PLABEL204" library="pinguin" package="PLABEL204" value="" x="29" y="38.5" smashed="yes" rot="MR0"/>
 </elements>
@@
 <wire x1="59.5" y1="42.5" x2="29.5" y2="42.5" width="0.6096" layer="16"/>
 <via x="29.5" y="42.5" extent="1-16" drill="0.35"/>
-<wire x1="20.080625" y1="40.38" x2="19.46" y2="40.38" width="0.6096" layer="1"/>
-<wire x1="21.437825" y1="41.7372" x2="20.080625" y2="40.38" width="0.6096" layer="1"/>
-<wire x1="29.5" y1="42.5" x2="28.7372" y2="41.7372" width="0.6096" layer="1"/>
-<wire x1="28.7372" y1="41.7372" x2="21.437825" y2="41.7372" width="0.6096" layer="1"/>
+<wire x1="20.937825" y1="42.7372" x2="19.46" y2="41.259375" width="0.6096" layer="1"/>
+<wire x1="19.46" y1="40.38" x2="19.46" y2="41.259375" width="0.6096" layer="1"/>
+<wire x1="29.5" y1="42.5" x2="29.2628" y2="42.7372" width="0.6096" layer="1"/>
+<wire x1="29.2628" y1="42.7372" x2="20.937825" y2="42.7372" width="0.6096" layer="1"/>
 <contactref element="KB2040-1" pad="4"/>
 <wire x1="73.13" y1="56.5" x2="75.87" y2="59.24" width="0.6096" layer="16"/>

Commit message: miso/mosi rev b
Connections:
- removed net MI: KB2040-2.3, TFT.6
- net MO: now also TFT.6; no longer TFT.7
Routing:
- net MI: track 28.1 -> 0.00 mm, vias 1 -> 0
- net MO: track 24.0 -> 25.1 mm
Changed lines of the file:
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@@
 <layer number="168" name="4mmHeightArea" color="7" fill="1" visible="no" active="yes"/>
 <layer number="170" name="Pinguin_tPlace" color="14" fill="1" visible="yes" active="yes"/>
-<layer number="171" name="Pinguin_bPlace" color="13" fill="1" visible="no" active="yes"/>
+<layer number="171" name="Pinguin_bPlace" color="13" fill="1" visible="yes" active="yes"/>
 <layer number="172" name="Pinguin_tBackup" color="14" fill="1" visible="no" active="yes"/>
 <layer number="173" name="Pinguin_bBackup" color="13" fill="1" visible="no" active="yes"/>
@@
 <wire x1="75.87" y1="41.87" x2="75.87" y2="44" width="0.6096" layer="1"/>
 </signal>
-<signal name="MI">
-<contactref element="KB2040-2" pad="3"/>
-<wire x1="68" y1="36" x2="73.5" y2="41.5" width="0.6096" layer="1"/>
-<wire x1="73.5" y1="41.5" x2="73.5" y2="43.83" width="0.6096" layer="1"/>
-<wire x1="73.5" y1="43.83" x2="73.33" y2="44" width="0.6096" layer="1"/>
-<wire x1="68" y1="36" x2="57.84" y2="36" width="0.6096" layer="1"/>
-<contactref element="TFT" pad="6"/>
-<via x="57.84" y="36" extent="1-16" drill="0.35"/>
-<wire x1="57.84" y1="36" x2="54" y2="36" width="0.6096" layer="16"/>
-<wire x1="54" y1="36" x2="52.3" y2="34.3" width="0.6096" layer="16"/>
-<wire x1="52.3" y1="34.3" x2="52.3" y2="33" width="0.6096" layer="16"/>
-</signal>
 <signal name="MO">
 <contactref element="KB2040-2" pad="2"/>
@@
 <wire x1="67" y1="37" x2="71" y2="41" width="0.6096" layer="1"/>
 <wire x1="71" y1="41" x2="71" y2="43.79" width="0.6096" layer="1"/>
-<contactref element="TFT" pad="7"/>
-<wire x1="56.3" y1="37" x2="54.84" y2="35.54" width="0.6096" layer="1"/>
-<wire x1="54.84" y1="35.54" x2="54.84" y2="33" width="0.6096" layer="1"/>
+<contactref element="TFT" pad="6"/>
+<wire x1="56.3" y1="37" x2="52.3" y2="33" width="0.6096" layer="1"/>
 </signal>
 <signal name="CS">
