File: TMC2209_Camera_Slider/PCB_Files/TMC2209_Camera_Slider_PCB_revB.sch (EAGLE design)
At the start: 14 parts, among them J1 1X2-3.5MM, J2 1X2-3.5MM, X1 REMBRANDT-ELECTRONICS---JST-X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, X2 REMBRANDT-ELECTRONICS---JST-X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

Commit message: miso/mosi rev b
Connections:
- removed net MI: KB2040-2.3, TFT.6
- net MO: now also TFT.6; no longer TFT.7
Changed lines of the file:
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@@
-</segment>
-</net>
-<net name="MI" class="0">
-<segment>
-<pinref part="KB2040-2" gate="G$1" pin="3"/>
-<wire x1="30.48" y1="50.8" x2="30.48" y2="60.96" width="0.1524" layer="91"/>
-<label x="30.48" y="58.42" size="1.778" layer="95" rot="R90"/>
-</segment>
-<segment>
-<pinref part="TFT" gate="G$1" pin="6"/>
-<wire x1="99.06" y1="30.48" x2="83.82" y2="30.48" width="0.1524" layer="91"/>
-<label x="83.82" y="30.48" size="1.778" layer="95"/>
 </segment>
 </net>
@@
 </segment>
 <segment>
-<pinref part="TFT" gate="G$1" pin="7"/>
-<wire x1="99.06" y1="27.94" x2="83.82" y2="27.94" width="0.1524" layer="91"/>
-<label x="83.82" y="27.94" size="1.778" layer="95"/>
+<pinref part="TFT" gate="G$1" pin="6"/>
+<wire x1="99.06" y1="30.48" x2="83.82" y2="30.48" width="0.1524" layer="91"/>
+<label x="83.82" y="30.48" size="1.778" layer="95"/>
 </segment>
 </net>

Commit message: tidy up schematic
clean up schematic for the motor slider learn guide
Other:
- note added: "JST Connectors"
- note added: "KB2040"
- note added: "Power"
- note added: "TFT"
- note added: "TMC2209 Breakouts"
- moved on the sheet: DCJACK, KB2040-1, KB2040-2, MOTOR1, MOTOR2, MPM3601, R1, R2, ROTARY, TFT, X1-1, X1-2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
